File: cad/cad_files/nav_control.sch (KiCad schematic (older format))
At the start: 10 parts

Commit message: Prep for layout (continued)
add footprints, refine design
Parts:
- added Rc102: 10k, SM0805, symbol R
- added Rc103: 10k, R4-LARGE_PADS, symbol R
- added THc101: 10k, symbol THERMISTOR
- added THc102: 10k, R4-LARGE_PADS, symbol THERMISTOR
- Rc101: footprint SM0805 -> R4-LARGE_PADS
Connections:
- wire segments 49 -> 59
- no-connect marks 18 -> 16
Changed lines of the file:
@@
-EESchema Schematic File Version 2  date Sun 07 Dec 2014 02:35:16 AM HST
+EESchema Schematic File Version 2  date Tue 09 Dec 2014 01:12:04 AM HST
 LIBS:local_parts
 LIBS:power
@@
 Sheet 2 4
 Title ""
-Date "7 dec 2014"
+Date "9 dec 2014"
 Rev ""
 Comp ""
@@
 Comment4 ""
 $EndDescr
+Connection ~ 1100 5800
+Wire Wire Line
+	1400 5700 1400 5800
+Wire Wire Line
+	1400 5800 1100 5800
+Connection ~ 1100 4300
+Wire Wire Line
+	1100 4300 1400 4300
+Wire Wire Line
+	1400 4300 1400 4400
+Connection ~ 1400 5100
+Wire Wire Line
+	2200 5100 1400 5100
+Connection ~ 1100 5000
+Wire Wire Line
+	1100 5200 1100 4900
+Connection ~ 2200 1100
+Wire Wire Line
+	2200 800  2200 1300
+Connection ~ 6400 2600
+Wire Wire Line
+	6700 2600 6200 2600
+Wire Wire Line
+	6200 2600 6200 2500
+Wire Wire Line
+	3800 5000 4000 5000
+Wire Wire Line
+	4600 2200 4500 2200
+Connection ~ 6600 2200
+Wire Wire Line
+	6600 2200 6600 2500
+Wire Wire Line
+	3800 4900 4000 4900
+Wire Wire Line
+	3800 4600 4000 4600
+Wire Wire Line
+	3800 4400 4000 4400
+Wire Wire Line
+	3100 6100 3100 6300
+Wire Wire Line
+	2900 3900 2900 3700
+Wire Wire Line
+	6600 2800 6600 2700
+Wire Wire Line
+	6600 2700 6700 2700
+Wire Wire Line
+	6600 2500 6700 2500
+Wire Wire Line
+	7100 2200 5500 2200
+Wire Wire Line
+	2200 1100 2000 1100
+Connection ~ 4500 1000
+Wire Wire Line
+	5600 1550 5600 1000
+Connection ~ 4100 2600
+Wire Wire Line
+	4100 2600 3300 2600
+Wire Wire Line
+	3300 2600 3300 2500
+Wire Wire Line
+	4500 2200 4500 1000
+Connection ~ 4100 1600
+Wire Wire Line
+	4100 2000 4100 1200
+Wire Wire Line
+	4100 1200 3900 1200
+Wire Wire Line
+	3900 1600 4100 1600
+Connection ~ 3300 1800
+Wire Wire Line
+	3100 1800 3300 1800
+Wire Wire Line
+	3300 2000 3300 1400
+Wire Wire Line
+	3300 1600 3500 1600
+Connection ~ 3300 1600
+Wire Wire Line
+	3300 1200 3500 1200
+Wire Wire Line
+	4100 1800 4300 1800
+Connection ~ 4100 1800
+Wire Wire Line
+	2300 1000 2300 1800
+Wire Wire Line
+	2300 1800 2500 1800
+Wire Wire Line
+	4100 2700 4100 2500
+Wire Wire Line
+	5600 2200 5600 2050
+Connection ~ 5600 2200
+Wire Wire Line
+	5600 1000 2000 1000
+Connection ~ 2300 1000
+Wire Wire Line
+	6400 2500 6400 2600
+Wire Wire Line
+	2900 3100 2900 3200
+Wire Wire Line
+	2700 3300 2700 3900
+Wire Wire Line
+	3200 6100 3200 6200
+Wire Wire Line
+	3200 6200 3100 6200
+Connection ~ 3100 6200
+Wire Wire Line
+	3800 4500 4000 4500
+Wire Wire Line
+	3800 4800 4000 4800
+Wire Wire Line
+	6400 2200 6400 2000
+Connection ~ 6400 2200
+Wire Wire Line
+	4300 1800 4300 2600
+Wire Wire Line
+	4300 2600 4600 2600
+Wire Wire Line
+	4600 2400 4500 2400
+Wire Wire Line
+	4500 2400 4500 2500
+Wire Wire Line
+	5500 2600 5600 2600
+Wire Wire Line
+	2500 1000 2500 800
+Connection ~ 2500 1000
+Wire Wire Line
+	2900 3800 3200 3800
+Wire Wire Line
+	3200 3800 3200 3700
+Connection ~ 2900 3800
+Wire Wire Line
+	1100 5000 2200 5000
+Wire Wire Line
+	1400 4900 1400 5200
+Wire Wire Line
+	1100 4200 1100 4400
+Wire Wire Line
+	1100 5900 1100 5700
+$Comp
+L THERMISTOR THc101
+U 1 1 54868248
+P 1100 5450
+F 0 "THc101" V 1200 5500 50  0000 C CNN
+F 1 "10k" V 1000 5450 50  0000 C CNN
+	1    1100 5450
+	1    0    0    -1
+$EndComp
+$Comp
+L R Rc102
+U 1 1 54868245
+P 1100 4650
+F 0 "Rc102" V 1180 4650 50  0000 C CNN
+F 1 "10k" V 1100 4650 50  0000 C CNN
+F 2 "SM0805" H 1100 4650 60  0001 C CNN
+	1    1100 4650
+	1    0    0    -1
+$EndComp
+$Comp
+L GND #PWR?
+U 1 1 54868229
+P 1100 5900
+F 0 "#PWR?" H 1100 5900 30  0001 C CNN
+F 1 "GND" H 1100 5830 30  0001 C CNN
+	1    1100 5900
+	1    0    0    -1
+$EndComp
+$Comp
+L +5V #PWR?
+U 1 1 54868223
+P 1100 4200
+F 0 "#PWR?" H 1100 4290 20  0001 C CNN
+F 1 "+5V" H 1100 4290 30  0000 C CNN
+	1    1100 4200
+	1    0    0    -1
+$EndComp
+$Comp
+L THERMISTOR THc102
+U 1 1 548681F5
+P 1400 5450
+F 0 "THc102" V 1500 5500 50  0000 C CNN
+F 1 "10k" V 1300 5450 50  0000 C CNN
+F 2 "R4-LARGE_PADS" H 1400 5450 60  0001 C CNN
+	1    1400 5450
+	1    0    0    -1
+$EndComp
+$Comp
+L R Rc103
+U 1 1 548681C7
+P 1400 4650
+F 0 "Rc103" V 1480 4650 50  0000 C CNN
+F 1 "10k" V 1400 4650 50  0000 C CNN
+F 2 "R4-LARGE_PADS" H 1400 4650 60  0001 C CNN
+	1    1400 4650
+	1    0    0    -1
+$EndComp
 Text Notes 4900 5100 0    60   ~ 0
 A0 / A1 thermistor or similar for monitoring \nLED temperature (maybe battery too)
-Connection ~ 2200 1100
-Wire Wire Line
-	2200 800  2200 1300
-Connection ~ 6400 2600
-Wire Wire Line
-	6700 2600 6200 2600
-Wire Wire Line
-	6200 2600 6200 2500
-Wire Wire Line
-	3800 5000 4000 5000
-Wire Wire Line
-	4600 2200 4500 2200
-Connection ~ 6600 2200
-Wire Wire Line
-	6600 2500 6600 2200
-Wire Wire Line
-	3800 4900 4000 4900
-Wire Wire Line
-	3800 4600 4000 4600
-Wire Wire Line
-	3800 4400 4000 4400
-Wire Wire Line
-	3100 6100 3100 6300
-Wire Wire Line
-	2900 3900 2900 3700
-Wire Wire Line
-	6600 2800 6600 2700
-Wire Wire Line
-	6600 2700 6700 2700
-Wire Wire Line
-	6600 2500 6700 2500
-Wire Wire Line
-	7100 2200 5500 2200
-Wire Wire Line
-	2200 1100 2000 1100
-Connection ~ 4500 1000
-Wire Wire Line
-	5600 1000 5600 1550
-Connection ~ 4100 2600
-Wire Wire Line
-	3300 2600 4100 2600
-Wire Wire Line
-	3300 2600 3300 2500
-Wire Wire Line
-	4500 2200 4500 1000
-Connection ~ 4100 1600
-Wire Wire Line
-	4100 2000 4100 1200
-Wire Wire Line
-	4100 1200 3900 1200
-Wire Wire Line
-	3900 1600 4100 1600
-Connection ~ 3300 1800
-Wire Wire Line
-	3100 1800 3300 1800
-Wire Wire Line
-	3300 2000 3300 1400
-Wire Wire Line
-	3300 1600 3500 1600
-Connection ~ 3300 1600
-Wire Wire Line
-	3300 1200 3500 1200
-Wire Wire Line
-	4100 1800 4300 1800
-Connection ~ 4100 1800
-Wire Wire Line
-	2300 1000 2300 1800
-Wire Wire Line
-	2300 1800 2500 1800
-Wire Wire Line
-	4100 2700 4100 2500
-Wire Wire Line
-	5600 2200 5600 2050
-Connection ~ 5600 2200
-Wire Wire Line
-	2000 1000 5600 1000
-Connection ~ 2300 1000
-Wire Wire Line
-	6400 2500 6400 2600
-Wire Wire Line
-	2900 3100 2900 3200
-Wire Wire Line
-	2700 3300 2700 3900
-Wire Wire Line
-	3200 6100 3200 6200
-Wire Wire Line
-	3200 6200 3100 6200
-Connection ~ 3100 6200
-Wire Wire Line
-	3800 4500 4000 4500
-Wire Wire Line
-	3800 4800 4000 4800
-Wire Wire Line
-	6400 2200 6400 2000
-Connection ~ 6400 2200
-Wire Wire Line
-	4300 1800 4300 2600
-Wire Wire Line
-	4300 2600 4600 2600
-Wire Wire Line
-	4600 2400 4500 2400
-Wire Wire Line
-	4500 2400 4500 2500
-Wire Wire Line
-	5500 2600 5600 2600
-Wire Wire Line
-	2500 1000 2500 800
-Connection ~ 2500 1000
-Wire Wire Line
-	2900 3800 3200 3800
-Wire Wire Line
-	3200 3800 3200 3700
-Connection ~ 2900 3800
 $Comp
 L PWR_FLAG #FLG01
@@
 NoConn ~ 2200 5300
 NoConn ~ 2200 5200
-NoConn ~ 2200 5100
-NoConn ~ 2200 5000
 NoConn ~ 2200 4800
 NoConn ~ 2200 4700
@@
 F 0 "Rc101" V 2980 3450 50  0000 C CNN
 F 1 "DNP" V 2900 3450 50  0000 C CNN
-F 2 "SM0805" H 2900 3450 60  0001 C CNN
+F 2 "R4-LARGE_PADS" H 2900 3450 60  0001 C CNN
 	1    2900 3450
 	1    0    0    -1
