File: cad/cad_files/nav_control.sch (KiCad schematic (older format))
At the start: 14 parts

Commit message: Bom updating (and schematic) for LED power
Parts:
- Dp301, Dp302: digikey (none) -> B340LB-FDICT-ND
- Rc101: digikey (none) -> JW50ZT0R00CT-ND
- Rc102, Rp301, Rp302: digikey (none) -> 1276-5742-1-ND
- Rc103: digikey (none) -> A105970CT-ND
- THc101: digikey (none) -> 541-1150-1-ND
- THc102: digikey (none) -> 615-1054-ND
Changed lines of the file:
@@
-EESchema Schematic File Version 2  date Wed 24 Dec 2014 07:01:58 AM HST
+EESchema Schematic File Version 2  date Wed 24 Dec 2014 07:52:56 AM HST
 LIBS:local_parts
 LIBS:power
@@
 F 1 "10k" V 900 5450 50  0000 C CNN
 F 2 "SM1206" V 1200 5450 60  0000 C CNN
+F 4 "541-1150-1-ND" V 800 5450 60  0000 C CNN "digikey"
 	1    1000 5450
 	1    0    0    -1
@@
 F 1 "10k" V 1000 4650 50  0000 C CNN
 F 2 "SM1206" V 1200 4650 60  0000 C CNN
+F 4 "1276-5742-1-ND" V 900 4650 60  0000 C CNN "digikey"
 	1    1000 4650
 	1    0    0    -1
@@
 F 0 "THc102" V 1500 5500 50  0000 C CNN
 F 1 "10k" V 1300 5450 50  0000 C CNN
-F 2 "R4-LARGE_PADS" V 1600 5450 60  0000 C CNN
+F 2 "R4-LARGE_PADS" V 1600 5400 60  0000 C CNN
+F 4 "615-1054-ND" V 1700 5450 60  0000 C CNN "digikey"
 	1    1400 5450
 	1    0    0    -1
@@
 F 0 "Rc103" V 1480 4650 50  0000 C CNN
 F 1 "10k" V 1400 4650 50  0000 C CNN
-F 2 "R4-LARGE_PADS" V 1600 4650 60  0000 C CNN
+F 2 "R4-LARGE_PADS" V 1600 4800 60  0000 C CNN
+F 4 "A105970CT-ND" V 1700 4800 60  0000 C CNN "digikey"
 	1    1400 4650
 	1    0    0    -1
@@
 F 1 "DNP" V 2900 3450 50  0000 C CNN
 F 2 "R4-LARGE_PADS" V 3050 3450 60  0000 C CNN
+F 4 "JW50ZT0R00CT-ND" V 2800 3450 60  0000 C CNN "digikey"
 	1    2900 3450
 	1    0    0    -1
@@
 F 1 "DIODE" H 3700 1100 40  0000 C CNN
 F 2 "DO-214AA" H 3700 1000 60  0000 C CNN
+F 4 "B340LB-FDICT-ND" H 3700 1350 60  0000 C CNN "digikey"
 	1    3700 1200
 	1    0    0    -1
@@
 F 1 "DIODE" H 3700 1500 40  0000 C CNN
 F 2 "DO-214AA" H 3700 1400 60  0000 C CNN
+F 4 "B340LB-FDICT-ND" H 3700 1300 60  0000 C CNN "digikey"
 	1    3700 1600
 	1    0    0    -1
@@
 F 1 "10k" V 4100 2250 50  0000 C CNN
 F 2 "SM1206" V 4300 2250 60  0000 C CNN
+F 4 "1276-5742-1-ND" V 3950 2050 60  0000 C CNN "digikey"
 	1    4100 2250
 	1    0    0    -1
@@
 F 1 "10k" V 3300 2250 50  0000 C CNN
 F 2 "SM1206" V 3500 2250 60  0000 C CNN
+F 4 "1276-5742-1-ND" V 3600 2050 60  0000 C CNN "digikey"
 	1    3300 2250
 	1    0    0    -1

Commit message: Rearranging a few tracks (on board)
Parts:
- Up301: digikey (none) -> FPF2103CT-ND
Changed lines of the file:
@@
-EESchema Schematic File Version 2  date Wed 24 Dec 2014 07:52:56 AM HST
+EESchema Schematic File Version 2  date Wed 24 Dec 2014 08:27:14 AM HST
 LIBS:local_parts
 LIBS:power
@@
 F 1 "FPF2100" H 5250 2500 60  0000 C CNN
 F 2 "SOT23-5" H 5250 2000 60  0000 C CNN
+F 4 "FPF2103CT-ND" H 5250 2400 60  0000 C CNN "digikey"
 	1    5250 2400
 	1    0    0    -1

Commit message: Change TH thermistor footprint
switch from ``resistor'' to ``pin header'' style footprints
Parts:
- Rc103: footprint R4-LARGE_PADS -> PIN_ARRAY_2X1
Changed lines of the file:
@@
-EESchema Schematic File Version 2  date Wed 24 Dec 2014 08:27:14 AM HST
+EESchema Schematic File Version 2  date Sat 27 Dec 2014 01:12:34 AM HST
 LIBS:local_parts
 LIBS:power
@@
 Sheet 2 4
 Title ""
-Date "24 dec 2014"
+Date "27 dec 2014"
 Rev ""
 Comp ""
@@
 F 0 "Rc103" V 1480 4650 50  0000 C CNN
 F 1 "10k" V 1400 4650 50  0000 C CNN
-F 2 "R4-LARGE_PADS" V 1600 4800 60  0000 C CNN
+F 2 "PIN_ARRAY_2X1" V 1600 4800 60  0000 C CNN
 F 4 "A105970CT-ND" V 1700 4800 60  0000 C CNN "digikey"
 	1    1400 4650

Commit message: Re-arranging LED section
Working over thermal spreading
Resizing refdes markings
Moving thermistors
Parts:
- THc102: footprint R4-LARGE_PADS -> R3-LARGE_PADS
Changed lines of the file:
@@
-EESchema Schematic File Version 2  date Sat 27 Dec 2014 01:12:34 AM HST
+EESchema Schematic File Version 2  date Sat 27 Dec 2014 01:34:47 AM HST
 LIBS:local_parts
 LIBS:power
@@
 F 0 "THc102" V 1500 5500 50  0000 C CNN
 F 1 "10k" V 1300 5450 50  0000 C CNN
-F 2 "R4-LARGE_PADS" V 1600 5400 60  0000 C CNN
+F 2 "R3-LARGE_PADS" V 1600 5400 60  0000 C CNN
 F 4 "615-1054-ND" V 1700 5450 60  0000 C CNN "digikey"
 	1    1400 5450

Commit message: Fix footprints for TH thermocouple & resistor
THc102 and Rc103 (near lower edge of board, HPLED, and ext led connector)
Parts:
- Rc103: footprint PIN_ARRAY_2X1 -> R3-LARGE_PADS
- THc102: footprint R3-LARGE_PADS -> PIN_ARRAY_2X1
Changed lines of the file:
@@
-EESchema Schematic File Version 2  date Mon 29 Dec 2014 02:15:58 AM HST
+EESchema Schematic File Version 2  date Mon 29 Dec 2014 02:23:30 AM HST
 LIBS:local_parts
 LIBS:power
@@
 F 0 "THc102" V 1500 5500 50  0000 C CNN
 F 1 "10k" V 1300 5450 50  0000 C CNN
-F 2 "R3-LARGE_PADS" V 1600 5400 60  0000 C CNN
+F 2 "PIN_ARRAY_2X1" V 1600 5400 60  0000 C CNN
 F 4 "615-1054-ND" V 1700 5450 60  0000 C CNN "digikey"
 	1    1400 5450
@@
 F 0 "Rc103" V 1480 4650 50  0000 C CNN
 F 1 "10k" V 1400 4650 50  0000 C CNN
-F 2 "PIN_ARRAY_2X1" V 1600 4800 60  0000 C CNN
+F 2 "R3-LARGE_PADS" V 1600 4800 60  0000 C CNN
 F 4 "A105970CT-ND" V 1700 4800 60  0000 C CNN "digikey"
 	1    1400 4650
