File: cad/cad_files/nav_charge.sch (KiCad schematic (older format))
At the start: 26 parts

Commit message: Prep for layout (continued)
add footprints, refine design
Parts:
- Dp101, Dp102: footprint (none) -> DO-216AA
- Dp103, Rp107, Rp108, Rp112, THp101, THp102: footprint (none) -> SM1206
- Lp101: footprint (none) -> SLF7045
- Qp101: footprint (none) -> SOT23_6
- Rp101, Rp102, Rp103, Rp104, Rp105, Rp106, Rp109, Rp110, Rp111: footprint SM0805 -> SM1206
Connections:
- wire segments 80 -> 107
Other:
- note added: "TODO: 3A, 1W, \n also for Dp101"
- moved on the sheet: Cp102, Dp101, Dp102, Dp103, Lp101, Qp101, Rp101, Rp102, Rp103

Commit message: Prep for layout (continued)
add footprints, refine design
Parts:
- Dp101, Dp102: footprint DO-216AA -> DO-214AA
- Qp102: footprint (none) -> SOT89
Changed lines of the file:
@@
-EESchema Schematic File Version 2  date Wed 10 Dec 2014 07:12:18 PM HST
+EESchema Schematic File Version 2  date Thu 11 Dec 2014 12:57:18 AM HST
 LIBS:local_parts
 LIBS:power
@@
 P 7600 3100
 F 0 "Qp102" H 7600 2950 60  0000 R CNN
-F 1 "FCX718" H 7600 3250 60  0000 R CNN
+F 1 "FCX718" H 7600 3200 60  0000 R CNN
+F 2 "SOT89" H 7500 3300 60  0000 C CNN
 	1    7600 3100
 	1    0    0    1
@@
 F 0 "Dp102" H 3300 2500 40  0000 C CNN
 F 1 "DIODE" H 3300 2300 40  0000 C CNN
-F 2 "DO-216AA" H 3300 2200 60  0000 C CNN
+F 2 "DO-214AA" H 3300 2200 60  0000 C CNN
 	1    3300 2400
 	0    -1   -1   0
@@
 F 0 "Dp101" H 2900 1900 40  0000 C CNN
 F 1 "DIODE" H 2900 1700 40  0000 C CNN
-F 2 "DO-216AA" H 2900 1600 60  0000 C CNN
+F 2 "DO-214AA" H 2900 1600 60  0000 C CNN
 	1    2900 1800
 	-1   0    0    1

Commit message: Prep for layout (continued)
Add footprints, refine design

add additional ``LED footprint'' (pin header)
Connections:
- wire segments 107 -> 80
Changed lines of the file:
@@
-EESchema Schematic File Version 2  date Thu 11 Dec 2014 12:57:18 AM HST
+EESchema Schematic File Version 2  date Thu 11 Dec 2014 02:09:55 AM HST
 LIBS:local_parts
 LIBS:power
@@
 	6000 3800 5900 3800
 Wire Wire Line
-	4200 4200 4200 4100
-Wire Wire Line
-	5900 1500 1500 1500
+	4200 4100 4200 4200
+Wire Wire Line
+	1500 1500 5900 1500
 Connection ~ 4200 5100
 Wire Wire Line
@@
 Connection ~ 7700 6500
 Wire Wire Line
-	7700 6600 7700 6500
-Wire Wire Line
-	7700 6500 7700 6400
-Wire Wire Line
-	4200 5800 4200 5900
-Wire Wire Line
-	4200 5900 4200 6000
-Wire Wire Line
-	4200 4700 4200 5100
-Wire Wire Line
-	4200 5100 4200 5300
+	7700 6600 7700 6400
+Wire Wire Line
+	4200 5800 4200 6000
+Wire Wire Line
+	4200 4700 4200 5300
 Connection ~ 1500 2000
 Wire Wire Line
-	4300 2000 4300 1800
+	4300 1800 4300 2000
 Wire Wire Line
 	4500 3100 4500 4500
 Connection ~ 7700 3500
 Wire Wire Line
-	7700 3500 7900 3500
+	7900 3500 7700 3500
 Connection ~ 6100 6500
 Wire Wire Line
@@
 Connection ~ 7700 5300
 Wire Wire Line
-	7700 5900 7700 5300
-Wire Wire Line
-	7700 5300 7700 5200
-Wire Wire Line
-	7700 5200 7700 5100
+	7700 5900 7700 5100
 Wire Wire Line
 	6600 5100 6700 5100
@@
 	6900 4300 7700 4300
 Wire Wire Line
-	7700 3600 7700 3500
-Wire Wire Line
-	7700 3500 7700 3400
-Wire Wire Line
-	7700 3400 7700 3300
+	7700 3600 7700 3300
 Connection ~ 5900 2300
 Wire Wire Line
-	5900 2300 5400 2300
+	5400 2300 5900 2300
 Wire Wire Line
 	5400 2300 5400 2400
 Wire Wire Line
-	5400 3500 5400 3600
-Wire Wire Line
-	5400 3600 5400 3800
+	5400 3500 5400 3800
 Wire Wire Line
 	5400 3800 5700 3800
@@
 	7600 2700 7700 2700
 Wire Wire Line
-	6900 3100 7000 3100
-Wire Wire Line
-	7000 3100 7400 3100
+	6900 3100 7400 3100
 Wire Wire Line
 	4500 3100 3600 3100
 Connection ~ 1700 2000
 Wire Wire Line
-	2700 3100 2900 3100
-Wire Wire Line
-	2900 3100 3100 3100
+	2700 3100 3100 3100
 Wire Wire Line
 	2200 2600 2200 2800
@@
 Connection ~ 2500 2000
 Wire Wire Line
-	2500 2000 2500 1800
+	2500 1800 2500 2000
 Wire Wire Line
 	2500 1800 2700 1800
@@
 Connection ~ 2200 2000
 Wire Wire Line
-	3600 2000 3300 2000
-Wire Wire Line
-	3300 2000 3100 2000
+	3600 2000 3100 2000
 Wire Wire Line
 	4300 1800 3100 1800
@@
 	6200 3100 6200 3900
 Wire Wire Line
-	5900 1500 5900 2300
-Wire Wire Line
-	5900 2300 5900 2400
-Wire Wire Line
-	5900 3500 5900 3800
-Wire Wire Line
-	5900 3800 5900 3900
+	5900 2400 5900 1500
+Wire Wire Line
+	5900 3500 5900 3900
 Wire Wire Line
 	5400 2900 5400 3100
@@
 	5100 4700 5200 4700
 Wire Wire Line
-	7700 2900 7700 2700
-Wire Wire Line
-	7700 2700 7700 2000
+	7700 2000 7700 2900
 Connection ~ 7700 2700
 Wire Wire Line
-	7700 4200 7700 4300
-Wire Wire Line
-	7700 4300 7700 4500
+	7700 4200 7700 4500
 Wire Wire Line
 	6600 4900 6800 4900
@@
 	5800 5700 5800 5900
 Wire Wire Line
-	5800 6400 5800 6500
-Wire Wire Line
-	5800 6500 6000 6500
-Wire Wire Line
-	6000 6500 6100 6500
-Wire Wire Line
-	6100 6500 6700 6500
-Wire Wire Line
-	6700 6500 7700 6500
+	5800 6500 5800 6400
+Wire Wire Line
+	7700 6500 5800 6500
 Connection ~ 6000 6500
 Wire Wire Line
@@
 Connection ~ 7700 5200
 Wire Wire Line
-	7700 2000 4300 2000
-Wire Wire Line
-	4300 2000 4200 2000
+	4200 2000 7700 2000
 Connection ~ 4300 2000
 Wire Wire Line
-	1500 3100 2200 3100
+	2200 3100 1500 3100
 Wire Wire Line
 	900  2200 1100 2200
@@
 	1100 2200 1100 2400
 Wire Wire Line
-	3800 4700 3800 4900
-Wire Wire Line
-	3800 4900 3800 5300
-Wire Wire Line
-	3800 4100 3800 4200
+	3800 4700 3800 5300
+Wire Wire Line
+	3800 4200 3800 4100
 Wire Wire Line
 	3800 5800 3800 5900
@@
 Connection ~ 3800 4900
 Wire Wire Line
-	2700 2000 2500 2000
-Wire Wire Line
-	2500 2000 2200 2000
-Wire Wire Line
-	2200 2000 1700 2000
-Wire Wire Line
-	1700 2000 1500 2000
-Wire Wire Line
-	1500 2000 900  2000
-Wire Wire Line
-	4200 4100 3800 4100
-Wire Wire Line
-	3800 4100 1500 4100
-Wire Wire Line
-	1500 4100 1500 3100
-Wire Wire Line
-	1500 3100 1500 2000
-Wire Wire Line
-	1500 2000 1500 1500
+	2700 2000 900  2000
+Wire Wire Line
+	1500 4100 4200 4100
+Wire Wire Line
+	1500 1500 1500 4100
 Connection ~ 1500 3100
 Connection ~ 3800 4100
@@
 	4900 2200 7900 2200
 $Comp
-L PWR_FLAG #FLG012
+L PWR_FLAG #FLG014
 U 1 1 547FD854
 P 6000 3700
-F 0 "#FLG012" H 6000 3795 30  0001 C CNN
+F 0 "#FLG014" H 6000 3795 30  0001 C CNN
 F 1 "PWR_FLAG" H 6000 3880 30  0000 C CNN
 	1    6000 3700
@@
 thm1
 $Comp
-L GND #PWR013
+L GND #PWR015
 U 1 1 53DB3075
 P 7700 6600
-F 0 "#PWR013" H 7700 6600 30  0001 C CNN
+F 0 "#PWR015" H 7700 6600 30  0001 C CNN
 F 1 "GND" H 7700 6530 30  0001 C CNN
 	1    7700 6600
@@
 $EndComp
 $Comp
-L GND #PWR014
+L GND #PWR016
 U 1 1 53DB304B
 P 4200 6000
-F 0 "#PWR014" H 4200 6000 30  0001 C CNN
+F 0 "#PWR016" H 4200 6000 30  0001 C CNN
 F 1 "GND" H 4200 5930 30  0001 C CNN
 	1    4200 6000
@@
 WHY!?
 $Comp
-L GND #PWR015
+L GND #PWR017
 U 1 1 53DA2C30
 P 5100 4800
-F 0 "#PWR015" H 5100 4800 30  0001 C CNN
+F 0 "#PWR017" H 5100 4800 30  0001 C CNN
 F 1 "GND" H 5100 4730 30  0001 C CNN
 	1    5100 4800
@@
 $EndComp
 $Comp
-L GND #PWR016
+L GND #PWR018
 U 1 1 53DA0DD7
 P 1100 2400
-F 0 "#PWR016" H 1100 2400 30  0001 C CNN
+F 0 "#PWR018" H 1100 2400 30  0001 C CNN
 F 1 "GND" H 1100 2330 30  0001 C CNN
 	1    1100 2400
@@
 $EndComp
 $Comp
-L GND #PWR017
+L GND #PWR019
 U 1 1 53DA0D36
 P 1700 2800
-F 0 "#PWR017" H 1700 2800 30  0001 C CNN
+F 0 "#PWR019" H 1700 2800 30  0001 C CNN
 F 1 "GND" H 1700 2730 30  0001 C CNN
 	1    1700 2800
@@
 $EndComp
 $Comp
-L GND #PWR018
+L GND #PWR020
 U 1 1 53DA0D33
 P 2200 2800
-F 0 "#PWR018" H 2200 2800 30  0001 C CNN
+F 0 "#PWR020" H 2200 2800 30  0001 C CNN
 F 1 "GND" H 2200 2730 30  0001 C CNN
 	1    2200 2800
@@
 $EndComp
 $Comp
-L GND #PWR019
+L GND #PWR021
 U 1 1 53DA0D2E
 P 3300 2800
-F 0 "#PWR019" H 3300 2800 30  0001 C CNN
+F 0 "#PWR021" H 3300 2800 30  0001 C CNN
 F 1 "GND" H 3300 2730 30  0001 C CNN
 	1    3300 2800

Commit message: Updates during layout
Parts:
- removed Rp108: 10k, SM1206, symbol R
- removed THp102: 103AT-2, SM1206, symbol THERMISTOR
- BTp101, BTp102: footprint (none) -> PIN_ARRAY_2X1
- Cp101, Cp102, Cp103: footprint SM0805 -> SM1206
- Dp101, Dp102: footprint DO-214AA -> DO-214AB
- THp101: footprint SM1206 -> PIN_ARRAY_2X1
- Up101: footprint SOIC_16n -> SOIC16_N
Connections:
- wire segments 80 -> 76
Other:
- note added: "SKIP: power path for charger voltage rail \n (rather than cutting load power \n while charging)"
- note added: "TODO: 2x1 0.1" header for batteries, \n mount to ??? w/ #2 screws (0.098" dia holes)\n"
- note removed: "TODO: power path for charger voltage rail \n (rather than cutting load power \n while charging)"
- moved on the sheet: Rp107, THp101
Changed lines of the file:
@@
-EESchema Schematic File Version 2  date Thu 11 Dec 2014 02:09:55 AM HST
+EESchema Schematic File Version 2  date Tue 16 Dec 2014 01:21:59 AM HST
 LIBS:local_parts
 LIBS:power
@@
 Sheet 3 4
 Title "Battery Charger"
-Date "11 dec 2014"
+Date "16 dec 2014"
 Rev ""
 Comp ""
@@
 Comment4 ""
 $EndDescr
+Text Notes 8100 4000 0    60   ~ 0
+TODO: 2x1 0.1" header for batteries, \n    mount to ??? w/ #2 screws (0.098" dia holes)\n
 Text Notes 3600 2400 0    60   ~ 0
 TODO: 3A, 1W, \n  also for Dp101
@@
 Connection ~ 4200 5100
 Wire Wire Line
-	5200 5100 4200 5100
+	4200 5100 5200 5100
 Connection ~ 7700 6500
 Wire Wire Line
@@
 	1100 2200 1100 2400
 Wire Wire Line
-	3800 4700 3800 5300
-Wire Wire Line
-	3800 4200 3800 4100
-Wire Wire Line
-	3800 5800 3800 5900
-Wire Wire Line
-	3800 5900 4200 5900
-Connection ~ 4200 5900
-Wire Wire Line
-	5200 4900 3800 4900
-Connection ~ 3800 4900
+	5200 4900 4200 4900
+Connection ~ 4200 4900
 Wire Wire Line
 	2700 2000 900  2000
@@
 	1500 1500 1500 4100
 Connection ~ 1500 3100
-Connection ~ 3800 4100
 Wire Wire Line
 	5400 3600 4900 3600
@@
 	4900 2200 7900 2200
 $Comp
-L PWR_FLAG #FLG014
+L PWR_FLAG #FLG08
 U 1 1 547FD854
 P 6000 3700
-F 0 "#FLG014" H 6000 3795 30  0001 C CNN
+F 0 "#FLG08" H 6000 3795 30  0001 C CNN
 F 1 "PWR_FLAG" H 6000 3880 30  0000 C CNN
 	1    6000 3700
@@
 Text HLabel 7900 2200 2    60   Output ~ 0
 charge_status
-Text Notes 8000 3700 0    60   ~ 0
-TODO: power path for charger voltage rail \n  (rather than cutting load power \n    while charging)
+Text Notes 8100 3700 0    60   ~ 0
+SKIP: power path for charger voltage rail \n  (rather than cutting load power \n    while charging)
 Text Label 3700 3100 0    60   ~ 0
 ICHG_d
@@
 thm1
 $Comp
-L GND #PWR015
+L GND #PWR09
 U 1 1 53DB3075
 P 7700 6600
-F 0 "#PWR015" H 7700 6600 30  0001 C CNN
+F 0 "#PWR09" H 7700 6600 30  0001 C CNN
 F 1 "GND" H 7700 6530 30  0001 C CNN
 	1    7700 6600
@@
 $EndComp
 $Comp
-L GND #PWR016
+L GND #PWR010
 U 1 1 53DB304B
 P 4200 6000
-F 0 "#PWR016" H 4200 6000 30  0001 C CNN
+F 0 "#PWR010" H 4200 6000 30  0001 C CNN
 F 1 "GND" H 4200 5930 30  0001 C CNN
 	1    4200 6000
@@
 WHY!?
 $Comp
-L GND #PWR017
+L GND #PWR011
 U 1 1 53DA2C30
 P 5100 4800
-F 0 "#PWR017" H 5100 4800 30  0001 C CNN
+F 0 "#PWR011" H 5100 4800 30  0001 C CNN
 F 1 "GND" H 5100 4730 30  0001 C CNN
 	1    5100 4800
@@
 F 0 "BTp102" H 7700 5000 50  0000 C CNN
 F 1 "BATTERY" H 7700 4610 50  0000 C CNN
+F 2 "PIN_ARRAY_2X1" H 7700 5100 60  0000 C CNN
 	1    7700 4800
 	0    1    1    0
@@
 F 0 "BTp101" H 7700 4100 50  0000 C CNN
 F 1 "BATTERY" H 7700 3710 50  0000 C CNN
+F 2 "PIN_ARRAY_2X1" H 7700 4200 60  0000 C CNN
 	1    7700 3900
 	0    1    1    0
@@
 F 0 "Cp103" H 5950 3400 50  0000 L CNN
 F 1 "1uF" H 5950 3200 50  0000 L CNN
-F 2 "SM0805" H 6200 3300 60  0000 C CNN
+F 2 "SM1206" H 6200 3300 60  0000 C CNN
 	1    5900 3300
 	1    0    0    -1
@@
 P 5900 4800
 F 0 "Up101" H 5900 4700 50  0000 C CNN
-F 1 "DS2712" H 5900 4900 50  0000 C CNN
-F 2 "SOIC_16n" H 5900 4800 50  0000 C CNN
+F 1 "DS2712" H 5900 5000 50  0000 C CNN
+F 2 "SOIC16_N" H 5900 4800 50  0000 C CNN
 F 3 "DOCUMENTATION" H 5900 4800 50  0001 C CNN
 	1    5900 4800
@@
 $EndComp
 $Comp
-L GND #PWR018
+L GND #PWR012
 U 1 1 53DA0DD7
 P 1100 2400
-F 0 "#PWR018" H 1100 2400 30  0001 C CNN
+F 0 "#PWR012" H 1100 2400 30  0001 C CNN
 F 1 "GND" H 1100 2330 30  0001 C CNN
 	1    1100 2400
@@
 $EndComp
 $Comp
-L GND #PWR019
+L GND #PWR013
 U 1 1 53DA0D36
 P 1700 2800
-F 0 "#PWR019" H 1700 2800 30  0001 C CNN
+F 0 "#PWR013" H 1700 2800 30  0001 C CNN
 F 1 "GND" H 1700 2730 30  0001 C CNN
 	1    1700 2800
@@
 $EndComp
 $Comp
-L GND #PWR020
+L GND #PWR014
 U 1 1 53DA0D33
 P 2200 2800
-F 0 "#PWR020" H 2200 2800 30  0001 C CNN
+F 0 "#PWR014" H 2200 2800 30  0001 C CNN
 F 1 "GND" H 2200 2730 30  0001 C CNN
 	1    2200 2800
@@
 $EndComp
 $Comp
-L GND #PWR021
+L GND #PWR015
 U 1 1 53DA0D2E
 P 3300 2800
-F 0 "#PWR021" H 3300 2800 30  0001 C CNN
+F 0 "#PWR015" H 3300 2800 30  0001 C CNN
 F 1 "GND" H 3300 2730 30  0001 C CNN
 	1    3300 2800
@@
 F 0 "Dp102" H 3300 2500 40  0000 C CNN
 F 1 "DIODE" H 3300 2300 40  0000 C CNN
-F 2 "DO-214AA" H 3300 2200 60  0000 C CNN
+F 2 "DO-214AB" H 3300 2200 60  0000 C CNN
 	1    3300 2400
 	0    -1   -1   0
@@
 F 0 "Dp101" H 2900 1900 40  0000 C CNN
 F 1 "DIODE" H 2900 1700 40  0000 C CNN
-F 2 "DO-214AA" H 2900 1600 60  0000 C CNN
+F 2 "DO-214AB" H 2900 1600 60  0000 C CNN
 	1    2900 1800
 	-1   0    0    1
@@
 F 0 "Cp102" H 2250 2500 50  0000 L CNN
 F 1 "0.1uF" H 2250 2300 50  0000 L CNN
-F 2 "SM0805" H 2400 2200 60  0000 C CNN
+F 2 "SM1206" H 2400 2200 60  0000 C CNN
 	1    2200 2400
 	1    0    0    -1
@@
 F 0 "Cp101" H 1750 2500 50  0000 L CNN
 F 1 "47uF" H 1750 2300 50  0000 L CNN
-F 2 "SM0805" H 1900 2200 60  0000 C CNN
+F 2 "SM1206" H 1900 2200 60  0000 C CNN
 	1    1700 2400
 	1    0    0    -1
@@
 battery_pos
 $Comp
-L R Rp108
-U 1 1 53D0E86F
+L R Rp107
+U 1 1 53D0E86D
 P 4200 4450
-F 0 "Rp108" V 4280 4450 50  0000 C CNN
+F 0 "Rp107" V 4280 4450 50  0000 C CNN
 F 1 "10k" V 4200 4450 50  0000 C CNN
 F 2 "SM1206" V 4350 4450 60  0000 C CNN
@@
 $EndComp
 $Comp
-L R Rp107
-U 1 1 53D0E86D
-P 3800 4450
-F 0 "Rp107" V 3880 4450 50  0000 C CNN
-F 1 "10k" V 3800 4450 50  0000 C CNN
-F 2 "SM1206" V 3950 4450 60  0000 C CNN
-	1    3800 4450
-	-1   0    0    1
-$EndComp
-$Comp
-L THERMISTOR THp102
-U 1 1 53D0E843
-P 4200 5550
-F 0 "THp102" V 4300 5600 50  0000 C CNN
-F 1 "103AT-2" V 4100 5550 50  0000 C CNN
-F 2 "SM1206" V 4400 5550 60  0000 C CNN
-	1    4200 5550
-	1    0    0    -1
-$EndComp
-$Comp
 L THERMISTOR THp101
 U 1 1 53D0E839
-P 3800 5550
-F 0 "THp101" V 3900 5600 50  0000 C CNN
-F 1 "103AT-2" V 3700 5550 50  0000 C CNN
-F 2 "SM1206" V 4000 5550 60  0000 C CNN
-	1    3800 5550
-	1    0    0    -1
-$EndComp
+P 4200 5550
+F 0 "THp101" V 4300 5600 50  0000 C CNN
+F 1 "103AT-2" V 4100 5550 50  0000 C CNN
+F 2 "PIN_ARRAY_2X1" V 4400 5550 60  0000 C CNN
+	1    4200 5550
+	1    0    0    -1
+$EndComp
