File: cad/cad_files/nav_light.sch (KiCad schematic (older format))
At the start: 5 parts

Commit message: BoM updating (adding to schematic)
Connections:
- net labels added: bat_neg
- wire segments 23 -> 28
Changed lines of the file:
@@
-EESchema Schematic File Version 2  date Wed 24 Dec 2014 03:57:46 AM HST
+EESchema Schematic File Version 2  date Wed 24 Dec 2014 07:01:58 AM HST
 LIBS:local_parts
 LIBS:power
@@
 Comment4 ""
 $EndDescr
-$Comp
-L MECH MECH104
-U 1 1 54942F24
-P 8450 3450
-F 0 "MECH104" H 8450 3400 60  0000 C CNN
-F 1 "MECH" H 8450 3500 60  0000 C CNN
-F 2 "mech_hole__2" H 8450 3300 60  0000 C CNN
-	1    8450 3450
-	1    0    0    -1
-$EndComp
-$Comp
-L MECH MECH103
-U 1 1 54942F1E
-P 8450 3150
-F 0 "MECH103" H 8450 3100 60  0000 C CNN
-F 1 "MECH" H 8450 3200 60  0000 C CNN
-F 2 "mech_hole__2" H 8450 3000 60  0000 C CNN
-	1    8450 3150
-	1    0    0    -1
-$EndComp
-$Comp
-L MECH MECH102
-U 1 1 54942F19
-P 8450 2850
-F 0 "MECH102" H 8450 2800 60  0000 C CNN
-F 1 "MECH" H 8450 2900 60  0000 C CNN
-F 2 "mech_hole__2" H 8450 2700 60  0000 C CNN
-	1    8450 2850
-	1    0    0    -1
-$EndComp
-$Comp
-L MECH MECH101
-U 1 1 54942F11
-P 8450 2550
-F 0 "MECH101" H 8450 2500 60  0000 C CNN
-F 1 "MECH" H 8450 2600 60  0000 C CNN
-F 2 "mech_hole__2" H 8450 2400 60  0000 C CNN
-	1    8450 2550
-	1    0    0    -1
-$EndComp
+Connection ~ 8900 3150
+Wire Wire Line
+	8900 2550 8900 3450
+Wire Wire Line
+	8900 3450 8750 3450
+Connection ~ 8900 2550
+Wire Wire Line
+	8900 2850 8750 2850
 Wire Wire Line
 	2300 2800 2500 2800
@@
 Wire Wire Line
 	2300 2600 2500 2600
+Wire Wire Line
+	9000 2550 8750 2550
+Wire Wire Line
+	8900 3150 8750 3150
+Connection ~ 8900 2850
+Text Label 9000 2550 0    60   ~ 0
+bat_neg
+Text Label 4400 2800 0    60   ~ 0
+bat_neg
+$Comp
+L MECH MECH104
+U 1 1 54942F24
+P 8450 3450
+F 0 "MECH104" H 8450 3400 60  0000 C CNN
+F 1 "MECH" H 8450 3500 60  0000 C CNN
+F 2 "mech_hole__2" H 8450 3300 60  0000 C CNN
+	1    8450 3450
+	1    0    0    -1
+$EndComp
+$Comp
+L MECH MECH103
+U 1 1 54942F1E
+P 8450 3150
+F 0 "MECH103" H 8450 3100 60  0000 C CNN
+F 1 "MECH" H 8450 3200 60  0000 C CNN
+F 2 "mech_hole__2" H 8450 3000 60  0000 C CNN
+	1    8450 3150
+	1    0    0    -1
+$EndComp
+$Comp
+L MECH MECH102
+U 1 1 54942F19
+P 8450 2850
+F 0 "MECH102" H 8450 2800 60  0000 C CNN
+F 1 "MECH" H 8450 2900 60  0000 C CNN
+F 2 "mech_hole__2" H 8450 2700 60  0000 C CNN
+	1    8450 2850
+	1    0    0    -1
+$EndComp
+$Comp
+L MECH MECH101
+U 1 1 54942F11
+P 8450 2550
+F 0 "MECH101" H 8450 2500 60  0000 C CNN
+F 1 "MECH" H 8450 2600 60  0000 C CNN
+F 2 "mech_hole__2" H 8450 2400 60  0000 C CNN
+	1    8450 2550
+	1    0    0    -1
+$EndComp
 $Comp
 L CONN_2 Pp101

Commit message: Add fiducial marks (as mech entities in schmatic)
Parts:
- added MECH5, MECH6, MECH7: MECH, fiducial, symbol MECH
Connections:
- no-connect marks 0 -> 3
Changed lines of the file:
@@
-EESchema Schematic File Version 2  date Sat 27 Dec 2014 01:34:47 AM HST
+EESchema Schematic File Version 2  date Mon 29 Dec 2014 01:53:40 AM HST
 LIBS:local_parts
 LIBS:power
@@
 Sheet 1 4
 Title ""
-Date "27 dec 2014"
+Date "29 dec 2014"
 Rev ""
 Comp ""
@@
 Comment4 ""
 $EndDescr
+NoConn ~ 8750 4650
+$Comp
+L MECH MECH7
+U 1 1 54A140B1
+P 8450 4650
+F 0 "MECH7" H 8450 4600 60  0000 C CNN
+F 1 "MECH" H 8450 4700 60  0000 C CNN
+F 2 "fiducial" H 8450 4500 60  0000 C CNN
+	1    8450 4650
+	1    0    0    -1
+$EndComp
+$Comp
+L MECH MECH6
+U 1 1 54A140A7
+P 8450 4350
+F 0 "MECH6" H 8450 4300 60  0000 C CNN
+F 1 "MECH" H 8450 4400 60  0000 C CNN
+F 2 "fiducial" H 8450 4200 60  0000 C CNN
+	1    8450 4350
+	1    0    0    -1
+$EndComp
+NoConn ~ 8750 4350
+NoConn ~ 8750 4050
+$Comp
+L MECH MECH5
+U 1 1 54A14065
+P 8450 4050
+F 0 "MECH5" H 8450 4000 60  0000 C CNN
+F 1 "MECH" H 8450 4100 60  0000 C CNN
+F 2 "fiducial" H 8450 3900 60  0000 C CNN
+	1    8450 4050
+	1    0    0    -1
+$EndComp
 Connection ~ 8900 3150
 Wire Wire Line

Commit message: Minor re-positioning and editing
Parts:
- added MECH8: MECH, logo-OSHW_3mm, symbol MECH
Connections:
- no-connect marks 3 -> 4
Changed lines of the file:
@@
-EESchema Schematic File Version 2  date Mon 29 Dec 2014 01:53:40 AM HST
+EESchema Schematic File Version 2  date Mon 29 Dec 2014 02:15:58 AM HST
 LIBS:local_parts
 LIBS:power
@@
 Comment4 ""
 $EndDescr
+NoConn ~ 8750 5250
+$Comp
+L MECH MECH8
+U 1 1 54A145DD
+P 8450 5250
+F 0 "MECH8" H 8450 5200 60  0000 C CNN
+F 1 "MECH" H 8450 5300 60  0000 C CNN
+F 2 "logo-OSHW_3mm" H 8450 5100 60  0000 C CNN
+	1    8450 5250
+	1    0    0    -1
+$EndComp
 NoConn ~ 8750 4650
 $Comp
